Commit message: add_controller_can_use_topic_to_control

File: agv_description/xacro/agv_base.gazebo.xacro (robot description, xacro)
@@ -1,88 +1,10 @@
 <?xml version="1.0"?>
-<robot name="agv" xmlns:xacro="http://www.ros.org/wiki/xacro">
-    <!-- PROPERTY LIST -->
-    <xacro:property name="M_PI" value="3.1415926"/>
-    <xacro:property name="base_length" value="0.20"/>
-    <xacro:property name="base_width" value="0.16"/>
-    <xacro:property name="base_height" value="0.16"/>
-    <xacro:property name="wheel_radius" value="0.06"/>
-    <xacro:property name="wheel_length" value="0.025"/>
-    <xacro:property name="wheel_joint_y" value="0.19"/>
-    <xacro:property name="wheel_joint_z" value="0.05"/>
-    <xacro:property name="caster_radius" value="0.015"/> <!-- wheel_radius - ( base_length/2 - wheel_joint_z) -->
-    <xacro:property name="caster_joint_x" value="0.18"/>
-    <!-- Defining the colors used in this robot -->
-    <material name="yellow">
-        <color rgba="1 0.4 0 1"/>
-    </material>
-    <material name="black">
-        <color rgba="0 0 0 0.95"/>
-    </material>
-    <material name="gray">
-        <color rgba="0.75 0.75 0.75 1"/>
-    </material>
-    <!-- Macro for robot wheel -->
-    <xacro:macro name="wheel" params="prefix reflect">
-        <joint name="${prefix}_wheel_joint" type="continuous">
-            <origin xyz="0 ${reflect*wheel_joint_y} ${-wheel_joint_z}" rpy="0 0 0"/>
-            <parent link="base_link"/>
-            <child link="${prefix}_wheel_link"/>
-            <axis xyz="0 1 0"/>
-        </joint>
-        <link name="${prefix}_wheel_link">
-            <visual>
-                <origin xyz="0 0 0" rpy="${M_PI/2} 0 0" />
-                <geometry>
-                    <mesh filename="package://agv_description/meshes/agvs_wheel.dae" scale="1.0 1.0 1.0"/>
-                </geometry>
-                <material name="gray" />
-            </visual>
-        </link>
-    </xacro:macro>
-    <!-- Macro for robot caster -->
-    <xacro:macro name="caster" params="prefix reflect">
-        <joint name="${prefix}_caster_joint" type="continuous">
-            <origin xyz="${reflect*caster_joint_x} 0 ${-(base_length/2 + caster_radius)}" rpy="0 0 0"/>
-            <parent link="base_link"/>
-            <child link="${prefix}_caster_link"/>
-            <axis xyz="0 1 0"/>
-        </joint>
-        <link name="${prefix}_caster_link">
-            <visual>
-                <origin xyz="0 0 0" rpy="0 0 0"/>
-                <geometry>
-                    <sphere radius="${caster_radius}" />
-                </geometry>
-                <material name="black" />
-            </visual>
-        </link>
-    </xacro:macro>
-    <xacro:macro name="mbot_base">
-        <link name="base_footprint">
-            <visual>
-                <origin xyz="0 0 0" rpy="0 0 0" />
-                <geometry>
-                    <box size="0.001 0.001 0.001" />
-                </geometry>
-            </visual>
-        </link>
-        <joint name="base_footprint_joint" type="fixed">
-            <origin xyz="0 0 -0.005" rpy="0 0 0" />
-            <parent link="base_footprint"/>
-            <child link="base_link" />
-        </joint>
-        <link name="base_link">
-            <visual>
-                <origin xyz="0 0 0" rpy="0 0 0" />
-                <geometry>
-                    <box size="${base_length} ${base_width} ${base_height}"/>
-                </geometry>
-                <material name="yellow" />
-            </visual>
-        </link>
-        <wheel prefix="left" reflect="-1"/>
-        <wheel prefix="right" reflect="1"/>
-        <caster prefix="front" reflect="-1"/>
-        <caster prefix="back" reflect="1"/>
-    </xacro:macro>
+<robot>
+    <gazebo>
+        <plugin name="ros_control" filename="libgazebo_ros_control.so">
+            <robotNamespace>/agvs</robotNamespace>
+            <controlPeriod>0.001</controlPeriod>
+            <robotSimType>gazebo_ros_control/DefaultRobotHWSim</robotSimType>
+        </plugin>
+    </gazebo>
 </robot>

File: agv_description/xacro/agv_base.urdf.xacro (robot description, xacro)
@@ -1,4 +1,5 @@
 <?xml version="1.0"?>
-<robot name="agv" xmlns:xacro="http://www.ros.org/wiki/xacro">
+<robot name="agvs" xmlns:xacro="http://www.ros.org/wiki/xacro">
+    <xacro:include filename="$(find agv_description)/xacro/agv_base.gazebo.xacro" />
     <!-- PROPERTY LIST -->
     <xacro:property name="M_PI" value="3.1415926"/>
@@ -15,4 +16,5 @@
     <xacro:property name="steer_joint_effort_limit" value="100.0" />
     <xacro:property name="steer_joint_velocity_limit" value="100.0" />
+    <xacro:property name="motor_wheel_mechanical_reduction" value="100.0" />
     <!-- Defining the colors used in this robot -->
     <material name="yellow">
@@ -31,20 +33,22 @@
                 <origin xyz="0 0 0" rpy="0 0 0" />
                 <geometry>
-                    <mesh filename="package://agv_description/meshes/motor_wheel.dae" scale="1.0 1.0 1.0"/>
+                    <mesh filename="package://agv_description/meshes/motor_wheel.dae"/>
                 </geometry>
-                <material name="gray" />
             </visual>
+            <gazebo reference="${prefix}_motor_wheel_link">
+                <material>Gazebo/Gray</material>
+            </gazebo>
+            <collision>
+                <origin xyz="0 0 0" rpy="0 0 0" />
+                <geometry>
+	                <mesh filename="package://agv_description/meshes/motor_wheel.dae"/>
+                </geometry>
+            </collision>
+            <inertial>
+                <mass value="1.0" />
+                <origin xyz="0 0 0" />
+                <inertia  ixx="1.0" ixy="0.0"  ixz="0.0"  iyy="1.0"  iyz="0.0"  izz="1.0" />
+            </inertial>
         </link>
-        <collision>
-            <origin xyz="0 0 0" rpy="0 0 0" />
-            <geometry>
-	            <mesh filename="package://agv_description/meshes/motor_wheel.dae" scale="1.0 1.0 1.0"/>
-            </geometry>
-        </collision>
-        <inertial>
-            <mass value="10" />
-            <origin xyz="0 0 0" />
-            <inertia  ixx="0.01" ixy="0.0"  ixz="0.0"  iyy="0.01"  iyz="0.0"  izz="0.01" />
-        </inertial>
         <joint name="${prefix}_motor_wheel_joint" type="continuous">
             <origin xyz="${x} ${y} ${z}" rpy="0 0 0"/>
@@ -55,24 +59,36 @@
             <joint_properties damping="${steer_joint_damping}" friction="{steer_joint_friction}"/>
         </joint>
+        <transmission name="${prefix}_motor_wheel_trans">
+            <type>transmission_interface/SimpleTransmission</type>
+            <joint name="${prefix}_motor_wheel_joint">
+                <hardwareInterface>EffortJointInterface</hardwareInterface>
+            </joint>
+            <actuator name="${prefix}_motor_joint_motor">
+                <hardwareInterface>EffortJointInterface</hardwareInterface>
+                <mechanicalReduction>${motor_wheel_mechanical_reduction}</mechanicalReduction>
+            </actuator>
+        </transmission>
         <link name="${prefix}_wheel_link">
             <visual>
                 <origin xyz="0 0 0" rpy="0 0 0" />
                 <geometry>
-                    <mesh filename="package://agv_description/meshes/agvs_wheel.dae" scale="1.0 1.0 1.0"/>
+                    <mesh filename="package://agv_description/meshes/agvs_wheel.dae"/>
                 </geometry>
-                <material name="gray" />
             </visual>
+            <gazebo reference="${prefix}_wheel_link">
+                <material>Gazebo/Gray</material>
+            </gazebo>
+            <collision>
+                <origin xyz="0 0 0" rpy="0 0 0" />
+                <geometry>
+	                <mesh filename="package://agv_description/meshes/agvs_wheel.dae"/>
+                </geometry>
+            </collision>
+            <inertial>
+                <mass value="1.250" />
+                <origin xyz="0 0 0" />
+                <inertia  ixx="1.0" ixy="0.0"  ixz="0.0"  iyy="1.0"  iyz="0.0"  izz="1.0" />
+            </inertial>
         </link>
-        <collision>
-            <origin xyz="0 0 0" rpy="0 0 0" />
-            <geometry>
-	            <mesh filename="package://agv_description/meshes/agvs_wheel.dae" scale="1.0 1.0 1.0"/>
-            </geometry>
-        </collision>
-        <inertial>
-            <mass value="1.250" />
-            <origin xyz="0 0 0" />
-            <inertia  ixx="0.0109375" ixy="0.0"  ixz="0.0"  iyy="0.021125"  iyz="0.0"  izz="0.0109375" />
-        </inertial>
         <joint name="${prefix}_wheel_joint" type="continuous">
             <origin xyz="0 0 0" rpy="0 0 ${M_PI}"/>
@@ -83,4 +99,14 @@
             <joint_properties damping="${wheel_joint_damping}" friction="{wheel_joint_friction}"/>
         </joint>
+        <transmission name="${prefix}_wheel_trans">
+            <type>transmission_interface/SimpleTransmission</type>
+            <joint name="${prefix}_wheel_joint">
+	            <hardwareInterface>VelocityJointInterface</hardwareInterface>
+            </joint>
+            <actuator name="${prefix}_wheel_joint_motor">
+	            <hardwareInterface>VelocityJointInterface</hardwareInterface>
+                <mechanicalReduction>${wheel_mechanical_reduction}</mechanicalReduction>
+            </actuator>
+        </transmission>
     </xacro:macro>
     <xacro:macro name="agv_base">
@@ -92,4 +118,9 @@
                 </geometry>
             </visual>
+            <inertial>
+                <mass value="1.250" />
+                <origin xyz="0 0 0" />
+                <inertia  ixx="1.0" ixy="0.0"  ixz="0.0"  iyy="1.0"  iyz="0.0"  izz="1.0" />
+            </inertial>
         </link>
         <joint name="base_footprint_joint" type="fixed">
@@ -104,7 +135,14 @@
                     <box size="${base_length} ${base_width} ${base_height}"/>
                 </geometry>
-                <material name="gray" />
             </visual>
+            <inertial>
+                <mass value="1.250" />
+                <origin xyz="0 0 0" />
+                <inertia  ixx="1.0" ixy="0.0"  ixz="0.0"  iyy="1.0"  iyz="0.0"  izz="1.0" />
+            </inertial>
         </link>
+        <gazebo reference="base_link">
+            <material>Gazebo/Gray</material>
+        </gazebo>
         <wheel prefix="front_right" x="0.8" y="1.6" z="-0.27"/>
         <wheel prefix="front_left" x="0.8" y="-1.6" z="-0.27"/>

Commit message: Add_navigation_but_wheel_motor_has_problem

File: agv_description/xacro/agv_base.gazebo.xacro (robot description, xacro)
@@ -1,17 +1,8 @@
 <?xml version="1.0"?>
 <robot>
-<!--
-    <gazebo>
-        <plugin name="ros_control" filename="libgazebo_ros_control.so">
-            <robotNamespace>/agvs</robotNamespace>
-            <controlPeriod>0.001</controlPeriod>
-            <robotSimType>gazebo_ros_control/DefaultRobotHWSim</robotSimType>
-        </plugin>
-    </gazebo>
--->
     <gazebo>
         <plugin name="agvs_wheel_controller" filename="libgazebo_ros_skid_steer_drive.so">
             <updateRate>100.0</updateRate>
-            <robotNamespace>/</robotNamespace>
+            <robotNamespace>/agvs_wheel</robotNamespace>
             <leftFrontJoint>front_left_wheel_joint</leftFrontJoint>
             <rightFrontJoint>front_right_wheel_joint</rightFrontJoint>
@@ -32,5 +23,5 @@
     </gazebo>
     <gazebo>
-        <plugin name="agvs_controller" filename="libgazebo_ros_skid_steer_drive.so">
+        <plugin name="agvs_motor_controller" filename="libgazebo_ros_skid_steer_drive.so">
             <updateRate>100.0</updateRate>
             <robotNamespace>/agvs_motor_wheel</robotNamespace>

File: agv_description/xacro/agv_base.urdf.xacro (robot description, xacro)
@@ -127,5 +127,5 @@
         </link>
         <joint name="${prefix}_wheel_joint" type="continuous">
-            <origin xyz="0 0 0" rpy="0 0 ${M_PI}"/>
+            <origin xyz="0 0 0" rpy="0 0 0"/>
             <parent link="${prefix}_motor_wheel_link"/>
             <child link="${prefix}_wheel_link"/>

Commit message: Finish_navigation_fix_teleop

File: agv_description/xacro/agv_base.gazebo.xacro (robot description, xacro)
@@ -23,4 +23,11 @@
     </gazebo>
     <gazebo>
+        <plugin name="gazebo_ros_control" filename="libgazebo_ros_control.so">
+            <robotNamespace>/agvs</robotNamespace>
+            <robotSimType>gazebo_ros_control/DefaultRobotHWSim</robotSimType>
+        </plugin>
+    </gazebo>
+<!--
+    <gazebo>
         <plugin name="agvs_motor_controller" filename="libgazebo_ros_skid_steer_drive.so">
             <updateRate>100.0</updateRate>
@@ -43,3 +50,4 @@
         </plugin>
     </gazebo>
+-->
 </robot>

File: agv_description/xacro/agv_base.urdf.xacro (robot description, xacro)
@@ -40,20 +40,4 @@
                     <selfCollide>false</selfCollide>
                 </geometry>
-                <surface>
-                    <friction>
-                        <ode>
-                            <kp>1000000.0</kp>
-                            <kd>100.0</kd>
-                            <mu1>1.5</mu1>
-                            <mu2>1.5</mu2>
-                        </ode>
-                    </friction>
-                    <contact>
-                        <ode>
-                            <min_depth>0.001</min_depth>
-                            <kp>1e9</kp>
-                        </ode>
-                    </contact>
-                </surface>
             </collision>
             <inertial>
@@ -78,8 +62,8 @@
             <type>transmission_interface/SimpleTransmission</type>
             <joint name="${prefix}_motor_wheel_joint">
-                <hardwareInterface>hardware_interface/VelocityJointInterface</hardwareInterface>
+                <hardwareInterface>hardware_interface/EffortJointInterface</hardwareInterface>
             </joint>
             <actuator name="${prefix}_motor_joint_motor">
-                <hardwareInterface>hardware_interface/VelocityJointInterface</hardwareInterface>
+                <hardwareInterface>hardware_interface/EffortJointInterface</hardwareInterface>
                 <mechanicalReduction>${motor_wheel_mechanical_reduction}</mechanicalReduction>
             </actuator>
@@ -101,20 +85,4 @@
                     <selfCollide>false</selfCollide>
                 </geometry>
-                <surface>
-                    <friction>
-                        <ode>
-                            <kp>1000000.0</kp>
-                            <kd>100.0</kd>
-                            <mu1>1.5</mu1>
-                            <mu2>1.5</mu2>
-                        </ode>
-                    </friction>
-                    <contact>
-                        <ode>
-                            <min_depth>0.001</min_depth>
-                            <kp>1e9</kp>
-                        </ode>
-                    </contact>
-                </surface>
             </collision>
             <inertial>
@@ -134,4 +102,5 @@
             <joint_properties damping="${wheel_joint_damping}" friction="{wheel_joint_friction}"/>
         </joint>
+<!--
         <transmission name="${prefix}_wheel_trans">
             <type>transmission_interface/SimpleTransmission</type>
@@ -144,4 +113,5 @@
             </actuator>
         </transmission>
+-->
     </xacro:macro>
     <!-- Macro for agv_base -->

File: agv_description/xacro/sensors/lidar_gazebo.xacro (robot description, xacro)
@@ -22,7 +22,7 @@
                 <mass value="0.1" />
                 <origin xyz="0 0 0" />
-                <inertia ixx="1.0" ixy="0.0" ixz="0.0"
-                         iyy="1.0" iyz="0.0"
-                         izz="1.0" />
+                <inertia ixx="0.0" ixy="0.0" ixz="0.0"
+                         iyy="0.0" iyz="0.0"
+                         izz="0.0" />
             </inertial>
         </link>
@@ -46,5 +46,5 @@
                     <range>
                       <min>0.10</min>
-                      <max>30</max>
+                      <max>100</max>
                       <resolution>0.01</resolution>
                     </range>

Commit message: Can_topic_control_to_navigation_but_speed_has_problem

File: agv_description/xacro/agv_base.gazebo.xacro (robot description, xacro)
@@ -28,26 +28,3 @@
         </plugin>
     </gazebo>
-<!--
-    <gazebo>
-        <plugin name="agvs_motor_controller" filename="libgazebo_ros_skid_steer_drive.so">
-            <updateRate>100.0</updateRate>
-            <robotNamespace>/agvs_motor_wheel</robotNamespace>
-            <leftFrontJoint>front_left_motor_wheel_joint</leftFrontJoint>
-            <rightFrontJoint>front_right_motor_wheel_joint</rightFrontJoint>
-            <leftRearJoint>back_left_motor_wheel_joint</leftRearJoint>
-            <rightRearJoint>back_right_motor_wheel_joint</rightRearJoint>
-            <wheelSeparation>0.4</wheelSeparation>
-            <wheelDiameter>0.215</wheelDiameter>
-            <robotBaseFrame>base_footprint</robotBaseFrame>
-            <torque>20</torque>
-            <topicName>cmd_vel</topicName>
-            <odometryFrame>odom</odometryFrame>
-            <odometryTopic>odom</odometryTopic>
-            <broadcastTF>true</broadcastTF>
-            <publishTf>true</publishTf>
-            <publishWheelTF>true</publishWheelTF>
-            <publishWheelJointState>true</publishWheelJointState>
-        </plugin>
-    </gazebo>
--->
 </robot>

File: agv_description/xacro/agv_base.urdf.xacro (robot description, xacro)
@@ -19,9 +19,4 @@
     <!-- Macro for whell -->
     <xacro:macro name="wheel" params="prefix x y z">
-        <!--
-        <gazebo>
-            <static>true</static>
-        </gazebo>
-        -->
         <link name="${prefix}_motor_wheel_link">
             <visual>
@@ -102,24 +97,7 @@
             <joint_properties damping="${wheel_joint_damping}" friction="{wheel_joint_friction}"/>
         </joint>
-<!--
-        <transmission name="${prefix}_wheel_trans">
-            <type>transmission_interface/SimpleTransmission</type>
-            <joint name="${prefix}_wheel_joint">
-	            <hardwareInterface>hardware_interface/VelocityJointInterface</hardwareInterface>
-            </joint>
-            <actuator name="${prefix}_wheel_joint_motor">
-	            <hardwareInterface>hardware_interface/VelocityJointInterface</hardwareInterface>
-                <mechanicalReduction>${wheel_mechanical_reduction}</mechanicalReduction>
-            </actuator>
-        </transmission>
--->
     </xacro:macro>
     <!-- Macro for agv_base -->
     <xacro:macro name="agv_base">
-        <!--
-        <gazebo>
-            <static>true</static>
-        </gazebo>
-        -->
         <!-- base_footprint is a fictitious link(frame) that is on the ground right below base_link
              origin, navigation stack depends on this frame -->
