Commit message: Update_README_and_agvs_topic_control

File: agv_description/xacro/agv_base.urdf.xacro (robot description, xacro)
@@ -7,14 +7,14 @@
     <xacro:property name="base_width" value="4"/>
     <xacro:property name="base_height" value="0.25"/>
-    <xacro:property name="wheel_joint_damping" value="1.0" />
-    <xacro:property name="wheel_joint_friction" value="1.0" />
+    <xacro:property name="wheel_joint_damping" value="0.0" />
+    <xacro:property name="wheel_joint_friction" value="0.0" />
     <xacro:property name="wheel_joint_effort_limit" value="10.0" />
     <xacro:property name="wheel_joint_velocity_limit" value="20.0" />
-    <xacro:property name="wheel_mechanical_reduction" value="100.0" />
-    <xacro:property name="steer_joint_damping" value="2.0" />
-    <xacro:property name="steer_joint_friction" value="1.0" />
+    <xacro:property name="wheel_mechanical_reduction" value="1.0" />
+    <xacro:property name="steer_joint_damping" value="0.0" />
+    <xacro:property name="steer_joint_friction" value="0.0" />
     <xacro:property name="steer_joint_effort_limit" value="10.0" />
     <xacro:property name="steer_joint_velocity_limit" value="10.0" />
-    <xacro:property name="motor_wheel_mechanical_reduction" value="100.0" />
+    <xacro:property name="motor_wheel_mechanical_reduction" value="1.0" />
     <!-- Macro for whell -->
     <xacro:macro name="wheel" params="prefix x y z">
@@ -38,8 +38,25 @@
                 <geometry>
 	                <mesh filename="package://agv_description/meshes/motor_wheel.dae" scale="1.0 1.0 1.0"/>
-                </geometry>
+                    <selfCollide>false</selfCollide>
+                </geometry>
+                <surface>
+                    <friction>
+                        <ode>
+                            <kp>1000000.0</kp>
+                            <kd>100.0</kd>
+                            <mu1>1.5</mu1>
+                            <mu2>1.5</mu2>
+                        </ode>
+                    </friction>
+                    <contact>
+                        <ode>
+                            <min_depth>0.001</min_depth>
+                            <kp>1e9</kp>
+                        </ode>
+                    </contact>
+                </surface>
             </collision>
             <inertial>
-                <mass value="10.0" />
+                <mass value="0.5" />
                 <origin xyz="0 0 0" />
                 <inertia  ixx="1.0" ixy="0.0" ixz="0.0"
@@ -82,8 +99,25 @@
                 <geometry>
 	                <mesh filename="package://agv_description/meshes/agvs_wheel.dae" scale="1.0 1.0 1.0"/>
-                </geometry>
+                    <selfCollide>false</selfCollide>
+                </geometry>
+                <surface>
+                    <friction>
+                        <ode>
+                            <kp>1000000.0</kp>
+                            <kd>100.0</kd>
+                            <mu1>1.5</mu1>
+                            <mu2>1.5</mu2>
+                        </ode>
+                    </friction>
+                    <contact>
+                        <ode>
+                            <min_depth>0.001</min_depth>
+                            <kp>1e9</kp>
+                        </ode>
+                    </contact>
+                </surface>
             </collision>
             <inertial>
-                <mass value="125.0" />
+                <mass value="2.0" />
                 <origin xyz="0 0 0" />
                 <inertia  ixx="1.0" ixy="0.0" ixz="0.0"
@@ -141,15 +175,32 @@
             </visual>
             <collision>
-               <origin xyz="0 0 0" rpy="0 0 0 " />
-               <geometry>
+                <origin xyz="0 0 0" rpy="0 0 0 " />
+                <geometry>
                     <box size="${base_length} ${base_width} ${base_height}"/>
-               </geometry>
+                    <selfCollide>false</selfCollide>
+                </geometry>
+                <surface>
+                    <friction>
+                        <ode>
+                            <kp>1000000.0</kp>
+                            <kd>100.0</kd>
+                            <mu1>1.5</mu1>
+                            <mu2>1.5</mu2>
+                        </ode>
+                    </friction>
+                    <contact>
+                        <ode>
+                            <min_depth>0.001</min_depth>
+                            <kp>1e9</kp>
+                        </ode>
+                    </contact>
+                </surface>
             </collision>
             <inertial>
-                <mass value="225.0" />
+                <mass value="0.1" />
                 <origin xyz="0 0 0" />
-                <inertia  ixx="1.0" ixy="0.0" ixz="0.0"
-                          iyy="1.0" iyz="0.0"
-                          izz="1.0" />
+                <inertia  ixx="0.0" ixy="0.0" ixz="0.0"
+                          iyy="0.0" iyz="0.0"
+                          izz="0.0" />
             </inertial>
         </link>

File: agv_description/xacro/sensors/lidar_gazebo.xacro (robot description, xacro)
@@ -22,7 +22,7 @@
                 <mass value="0.1" />
                 <origin xyz="0 0 0" />
-                <inertia ixx="0.01" ixy="0.0" ixz="0.0"
-                         iyy="0.01" iyz="0.0"
-                         izz="0.01" />
+                <inertia ixx="1.0" ixy="0.0" ixz="0.0"
+                         iyy="1.0" iyz="0.0"
+                         izz="1.0" />
             </inertial>
         </link>

Commit message: change_map_and_wheel_motor

File: agv_description/xacro/agv_base.urdf.xacro (robot description, xacro)
@@ -22,6 +22,11 @@
             <visual>
                 <origin xyz="0 0 0" rpy="0 0 0" />
+                <!--
                 <geometry>
                     <mesh filename="package://agv_description/meshes/motor_wheel.dae" scale="1.0 1.0 1.0"/>
+                </geometry>
+                -->
+                <geometry>
+                    <box size="0.1 0.1 0.1" />
                 </geometry>
             </visual>
@@ -31,7 +36,11 @@
             <collision>
                 <origin xyz="0 0 0" rpy="0 0 0" />
+                <!--
                 <geometry>
-	                <mesh filename="package://agv_description/meshes/motor_wheel.dae" scale="1.0 1.0 1.0"/>
-                    <selfCollide>false</selfCollide>
+                    <mesh filename="package://agv_description/meshes/motor_wheel.dae" scale="1.0 1.0 1.0"/>
+                </geometry>
+                -->
+                <geometry>
+                    <box size="0.1 0.1 0.1" />
                 </geometry>
             </collision>

Commit message: Avoidance_has_some_problem_at_edge_of_horizon

File: agv_description/xacro/agv_base.urdf.xacro (robot description, xacro)
@@ -7,4 +7,14 @@
     <xacro:property name="base_width" value="4"/>
     <xacro:property name="base_height" value="0.25"/>
+    <xacro:property name="base_mass" value="250.0"/>
+    <xacro:property name="imu_size" value="0.001"/>
+    <xacro:property name="imu_height" value="0.001"/>
+    <xacro:property name="motor_length" value="0.05"/>
+    <xacro:property name="motor_width" value="0.05"/>
+    <xacro:property name="motor_height" value="0.05"/>
+    <xacro:property name="motor_mass" value="20.0"/>
+    <xacro:property name="wheel_radius" value="0.05"/>
+    <xacro:property name="wheel_width" value="0.05"/>
+    <xacro:property name="wheel_mass" value="10.0" />
     <xacro:property name="wheel_joint_damping" value="0.0" />
     <xacro:property name="wheel_joint_friction" value="0.0" />
@@ -28,5 +38,5 @@
                 -->
                 <geometry>
-                    <box size="0.1 0.1 0.1" />
+                    <box size="${motor_length} ${motor_width} ${motor_height}" />
                 </geometry>
             </visual>
@@ -42,14 +52,10 @@
                 -->
                 <geometry>
-                    <box size="0.1 0.1 0.1" />
+                    <box size="${motor_length} ${motor_width} ${motor_height}" />
                 </geometry>
             </collision>
-            <inertial>
-                <mass value="0.5" />
-                <origin xyz="0 0 0" />
-                <inertia  ixx="1.0" ixy="0.0" ixz="0.0"
-                          iyy="1.0" iyz="0.0"
-                          izz="1.0" />
-            </inertial>
+            <xacro:box_inertial mass="${motor_mass}" x="${motor_length}" y="${motor_width}" z="${motor_height}">
+                <origin xyz="0 0 0" rpy="0 0 0" />
+            </xacro:box_inertial>
         </link>
         <joint name="${prefix}_motor_wheel_joint" type="continuous">
@@ -75,7 +81,10 @@
         <link name="${prefix}_wheel_link">
             <visual>
-                <origin xyz="0 0 0" rpy="0 0 0" />
+                <origin xyz="0 0 0" rpy="${0.5 * M_PI} 0 0" />
                 <geometry>
+                    <cylinder length="${wheel_width}" radius="${wheel_radius}"/>
+                <!--
                     <mesh filename="package://agv_description/meshes/agvs_wheel.dae" scale="1.0 1.0 1.0"/>
+                -->
                 </geometry>
 	            <material name="red">
@@ -84,20 +93,27 @@
             </visual>
             <collision>
-                <origin xyz="0 0 0" rpy="0 0 0" />
+                <origin xyz="0 0 0" rpy="${0.5 * M_PI} 0 0" />
                 <geometry>
-	                <mesh filename="package://agv_description/meshes/agvs_wheel.dae" scale="1.0 1.0 1.0"/>
+                    <cylinder length="${wheel_width}" radius="${wheel_radius}"/>
+	            <!--
+                    <mesh filename="package://agv_description/meshes/agvs_wheel.dae" scale="1.0 1.0 1.0"/>
                     <selfCollide>false</selfCollide>
+                -->
                 </geometry>
+                <friction>
+                    <ode>
+                        <mu>1.0</mu>
+                        <mu2>0.0</mu2>
+                        <slip1>1.0</slip1>
+                        <slip2>1.0</slip2>
+                    </ode>
+                </friction>
             </collision>
-            <inertial>
-                <mass value="2.0" />
-                <origin xyz="0 0 0" />
-                <inertia  ixx="1.0" ixy="0.0" ixz="0.0"
-                          iyy="1.0" iyz="0.0"
-                          izz="1.0" />
-            </inertial>
+            <xacro:cylinder_inertial mass="${wheel_mass}" radius="${wheel_radius}" length="${wheel_width}">
+                <origin xyz="0 0 0" rpy="${0.5 * M_PI} 0 0" />
+            </xacro:cylinder_inertial>
         </link>
         <joint name="${prefix}_wheel_joint" type="continuous">
-            <origin xyz="0 0 0" rpy="0 0 0"/>
+            <origin xyz="0 0 -0.075" rpy="0 0 0"/>
             <parent link="${prefix}_motor_wheel_link"/>
             <child link="${prefix}_wheel_link"/>
@@ -106,4 +122,22 @@
             <joint_properties damping="${wheel_joint_damping}" friction="{wheel_joint_friction}"/>
         </joint>
+    </xacro:macro>
+    <xacro:macro name="cylinder_inertial" params="radius length mass *origin">
+        <inertial>
+        <mass value="${mass}" />
+        <xacro:insert_block name="origin" />
+        <inertia ixx="${0.0833333 * mass * (3 * radius * radius + length * length)}" ixy="0.0" ixz="0.0"
+            iyy="${0.0833333 * mass * (3 * radius * radius + length * length)}" iyz="0.0"
+            izz="${0.5 * mass * radius * radius}" />
+        </inertial>
+    </xacro:macro>
+    <xacro:macro name="box_inertial" params="x y z mass *origin">
+        <inertial>
+        <mass value="${mass}" />
+        <xacro:insert_block name="origin" />
+        <inertia ixx="${0.0833333 * mass * (y*y + z*z)}" ixy="0.0" ixz="0.0"
+            iyy="${0.0833333 * mass * (x*x + z*z)}" iyz="0.0"
+            izz="${0.0833333 * mass * (x*x + y*y)}" />
+        </inertial>
     </xacro:macro>
     <!-- Macro for agv_base -->
@@ -120,5 +154,5 @@
         </link>
         <joint name="base_joint" type="fixed">
-            <origin xyz="0 0 0.394815" rpy="0 0 0" />
+            <origin xyz="0 0 0.275" rpy="0 0 0" />
             <parent link="base_footprint"/>
             <child link="base_link" />
@@ -135,38 +169,23 @@
                 <geometry>
                     <box size="${base_length} ${base_width} ${base_height}"/>
-                    <selfCollide>false</selfCollide>
                 </geometry>
-                <surface>
-                    <friction>
-                        <ode>
-                            <kp>1000000.0</kp>
-                            <kd>100.0</kd>
-                            <mu1>1.5</mu1>
-                            <mu2>1.5</mu2>
-                        </ode>
-                    </friction>
-                    <contact>
-                        <ode>
-                            <min_depth>0.001</min_depth>
-                            <kp>1e9</kp>
-                        </ode>
-                    </contact>
-                </surface>
             </collision>
-            <inertial>
-                <mass value="0.1" />
-                <origin xyz="0 0 0" />
-                <inertia  ixx="0.0" ixy="0.0" ixz="0.0"
-                          iyy="0.0" iyz="0.0"
-                          izz="0.0" />
-            </inertial>
+            <xacro:box_inertial mass="${base_mass}" x="${base_length}" y="${base_width}" z="${base_height}">
+                <origin xyz="0 0 0" rpy="0 0 0" />
+            </xacro:box_inertial>
         </link>
         <gazebo reference="base_link">
             <material>Gazebo/Gray</material>
         </gazebo>
+<!--
         <wheel prefix="front_right" x=" 0.8"  y=" 1.6" z="-0.285"/>
         <wheel prefix="front_left"  x=" 0.8"  y="-1.6" z="-0.285"/>
         <wheel prefix="back_right"  x="-0.8"  y=" 1.6" z="-0.285"/>
         <wheel prefix="back_left"   x="-0.8"  y="-1.6" z="-0.285"/>
+-->
+        <wheel prefix="front_right" x=" 0.8"  y=" 1.6" z="-0.15"/>
+        <wheel prefix="front_left"  x=" 0.8"  y="-1.6" z="-0.15"/>
+        <wheel prefix="back_right"  x="-0.8"  y=" 1.6" z="-0.15"/>
+        <wheel prefix="back_left"   x="-0.8"  y="-1.6" z="-0.15"/>
     </xacro:macro>
 </robot>

File: agv_description/xacro/goods/goods_gazebo.xacro (robot description, xacro)
@@ -3,4 +3,33 @@
     <!-- PROPERTY LIST -->
     <xacro:property name="M_PI" value="3.14159265359"/>
+    <xacro:property name="my_7m_goods_length" value="2.5"/>
+    <xacro:property name="my_7m_goods_width" value="7.0"/>
+    <xacro:property name="my_7m_goods_height" value="0.1"/>
+    <xacro:property name="my_7m_goods_mass" value="500.0"/>
+    <xacro:property name="legs_length" value="0.15"/>
+    <xacro:property name="legs_width" value="0.15"/>
+    <xacro:property name="legs_height" value="0.15"/>
+    <xacro:property name="legs_mass" value="10.0"/>
+    <xacro:property name="pillar_radius" value="0.1"/>
+    <xacro:property name="pillar_width" value="0.05"/>
+    <xacro:property name="pillar_mass" value="10.0" />
+    <xacro:macro name="cylinder_inertial" params="radius length mass *origin">
+        <inertial>
+        <mass value="${mass}" />
+        <xacro:insert_block name="origin" />
+        <inertia ixx="${0.0833333 * mass * (3 * radius * radius + length * length)}" ixy="0.0" ixz="0.0"
+            iyy="${0.0833333 * mass * (3 * radius * radius + length * length)}" iyz="0.0"
+            izz="${0.5 * mass * radius * radius}" />
+        </inertial>
+    </xacro:macro>
+    <xacro:macro name="box_inertial" params="x y z mass *origin">
+        <inertial>
+        <mass value="${mass}" />
+        <xacro:insert_block name="origin" />
+        <inertia ixx="${0.0833333 * mass * (y*y + z*z)}" ixy="0.0" ixz="0.0"
+            iyy="${0.0833333 * mass * (x*x + z*z)}" iyz="0.0"
+            izz="${0.0833333 * mass * (x*x + y*y)}" />
+        </inertial>
+    </xacro:macro>
     <xacro:macro name="legs" params="prefix x y z">
         <!-- Create laser reference frame -->
@@ -9,5 +38,5 @@
                 <origin xyz=" 0 0 0 " rpy="0 0 0" />
                 <geometry>
-                    <box size="0.15 0.15 0.15" />
+                    <box size="${legs_length} ${legs_width} ${legs_height}" />
                 </geometry>
                 <material name="black"/>
@@ -16,14 +45,10 @@
                 <origin xyz=" 0 0 0 " rpy="0 0 0" />
                 <geometry>
-                    <box size="0.15 0.15 0.15" />
+                    <box size="${legs_length} ${legs_width} ${legs_height}" />
                 </geometry>
             </collision>
-            <inertial>
-                <mass value="0.1" />
-                <origin xyz="0 0 0" />
-                <inertia ixx="1.0" ixy="0.0" ixz="0.0"
-                         iyy="1.0" iyz="0.0"
-                         izz="1.0" />
-            </inertial>
+            <xacro:box_inertial mass="${legs_mass}" x="${legs_length}" y="${legs_width}" z="${legs_height}">
+                <origin xyz="0 0 0" rpy="0 0 0" />
+            </xacro:box_inertial>
         </link>
         <joint name="${prefix}_leg_joint" type="fixed">
@@ -42,5 +67,5 @@
                 <origin xyz=" 0 0 0 " rpy="0 0 0" />
                 <geometry>
-                    <cylinder length="0.05" radius="0.1"/>
+                    <cylinder length="${pillar_width}" radius="${pillar_radius}"/>
                 </geometry>
                 <material name="black"/>
@@ -49,14 +74,10 @@
                 <origin xyz=" 0 0 0 " rpy="0 0 0" />
                 <geometry>
-                    <cylinder length="0.05" radius="0.1"/>
+                    <cylinder length="${pillar_width}" radius="${pillar_radius}"/>
                 </geometry>
             </collision>
-            <inertial>
-                <mass value="0.1" />
-                <origin xyz="0 0 0" />
-                <inertia ixx="1.0" ixy="0.0" ixz="0.0"
-                         iyy="1.0" iyz="0.0"
-                         izz="1.0" />
-            </inertial>
+            <xacro:cylinder_inertial mass="${pillar_mass}" radius="${pillar_radius}" length="${pillar_width}">
+                <origin xyz="0 0 0" rpy="0 0 0" />
+            </xacro:cylinder_inertial>
         </link>
         <joint name="${prefix}_pillar_joint" type="fixed">
@@ -75,5 +96,5 @@
                 <origin xyz=" 0 0 0 " rpy="0 0 0" />
                 <geometry>
-                    <box size="2.5 7 0.1" />
+                    <box size="${my_7m_goods_length} ${my_7m_goods_width} ${my_7m_goods_height}" />
                 </geometry>
                 <material name="gray"/>
@@ -82,14 +103,10 @@
                 <origin xyz=" 0 0 0 " rpy="0 0 0" />
                 <geometry>
-                    <box size="2.5 7 0.1" />
+                    <box size="${my_7m_goods_length} ${my_7m_goods_width} ${my_7m_goods_height}" />
                 </geometry>
             </collision>
-            <inertial>
-                <mass value="0.1" />
-                <origin xyz="0 0 0" />
-                <inertia ixx="1.0" ixy="0.0" ixz="0.0"
-                         iyy="1.0" iyz="0.0"
-                         izz="1.0" />
-            </inertial>
+            <xacro:box_inertial mass="${my_7m_goods_mass}" x="${my_7m_goods_length}" y="${my_7m_goods_width}" z="${my_7m_goods_height}">
+                <origin xyz="0 0 0" rpy="0 0 0" />
+            </xacro:box_inertial>
         </link>
         <gazebo reference="7m_goods_link">

File: agv_description/xacro/sensors/lidar_gazebo.xacro (robot description, xacro)
@@ -33,5 +33,5 @@
             <sensor type="ray" name="rplidar">
                 <pose>0 0 0 0 0 0</pose>
-                <visualize>true</visualize>
+                <visualize>false</visualize>
                 <update_rate>5</update_rate>
                 <ray>
