Commit message: Fix_gazebo_drift_bug_and_add_worlds_goods_lidar_control_node

File: agv_description/xacro/agv.xacro (robot description, xacro)
@@ -2,4 +2,28 @@
 <robot name="arm" xmlns:xacro="http://www.ros.org/wiki/xacro">
     <xacro:include filename="$(find agv_description)/xacro/agv_base.urdf.xacro" />
+    <xacro:include filename="$(find agv_description)/xacro/sensors/lidar_gazebo.xacro" />
+    <xacro:include filename="$(find agv_description)/xacro/goods/goods_gazebo.xacro" />
+    <!-- property for lidar -->
+    <xacro:property name="lidar_offset_x" value="0" />
+    <xacro:property name="lidar_offset_y" value="0" />
+    <xacro:property name="lidar_offset_z" value="0.15" />
     <agv_base/>
+    <!-- lidar -->
+    <joint name="lidar_joint" type="fixed">
+        <origin xyz="${lidar_offset_x} ${lidar_offset_y} ${lidar_offset_z}" rpy="0 0 0" />
+        <parent link="base_link"/>
+        <child link="laser_link"/>
+    </joint>
+    <xacro:rplidar prefix="laser"/>
+    <!-- property for goods -->
+    <xacro:property name="goods_offset_x" value="0" />
+    <xacro:property name="goods_offset_y" value="0" />
+    <xacro:property name="goods_offset_z" value="0.215" />
+    <!-- goods -->
+    <joint name="goods_joint" type="fixed">
+        <origin xyz="${goods_offset_x} ${goods_offset_y} ${goods_offset_z}" rpy="0 0 0" />
+        <parent link="base_link"/>
+        <child link="7m_goods_link"/>
+    </joint>
+    <put_7m_goods/>
 </robot>

File: agv_description/xacro/agv_base.urdf.xacro (robot description, xacro)
@@ -3,5 +3,5 @@
     <xacro:include filename="$(find agv_description)/xacro/agv_base.gazebo.xacro" />
     <!-- PROPERTY LIST -->
-    <xacro:property name="M_PI" value="3.1415926"/>
+    <xacro:property name="M_PI" value="3.14159265359"/>
     <xacro:property name="base_length" value="2"/>
     <xacro:property name="base_width" value="4"/>
@@ -9,29 +9,24 @@
     <xacro:property name="wheel_joint_damping" value="1.0" />
     <xacro:property name="wheel_joint_friction" value="1.0" />
-    <xacro:property name="wheel_joint_effort_limit" value="1000.0" />
-    <xacro:property name="wheel_joint_velocity_limit" value="2000.0" />
-    <xacro:property name="wheel_mechanical_reduction" value="1.0" />
+    <xacro:property name="wheel_joint_effort_limit" value="10.0" />
+    <xacro:property name="wheel_joint_velocity_limit" value="20.0" />
+    <xacro:property name="wheel_mechanical_reduction" value="100.0" />
     <xacro:property name="steer_joint_damping" value="2.0" />
     <xacro:property name="steer_joint_friction" value="1.0" />
-    <xacro:property name="steer_joint_effort_limit" value="100.0" />
-    <xacro:property name="steer_joint_velocity_limit" value="100.0" />
+    <xacro:property name="steer_joint_effort_limit" value="10.0" />
+    <xacro:property name="steer_joint_velocity_limit" value="10.0" />
     <xacro:property name="motor_wheel_mechanical_reduction" value="100.0" />
-    <!-- Defining the colors used in this robot -->
-    <material name="yellow">
-        <color rgba="1 0.4 0 1"/>
-    </material>
-    <material name="black">
-        <color rgba="0 0 0 0.95"/>
-    </material>
-    <material name="gray">
-        <color rgba="0.75 0.75 0.75 1"/>
-    </material>
     <!-- Macro for whell -->
     <xacro:macro name="wheel" params="prefix x y z">
+        <!--
+        <gazebo>
+            <static>true</static>
+        </gazebo>
+        -->
         <link name="${prefix}_motor_wheel_link">
             <visual>
                 <origin xyz="0 0 0" rpy="0 0 0" />
                 <geometry>
-                    <mesh filename="package://agv_description/meshes/motor_wheel.dae"/>
+                    <mesh filename="package://agv_description/meshes/motor_wheel.dae" scale="1.0 1.0 1.0"/>
                 </geometry>
             </visual>
@@ -42,11 +37,13 @@
                 <origin xyz="0 0 0" rpy="0 0 0" />
                 <geometry>
-	                <mesh filename="package://agv_description/meshes/motor_wheel.dae"/>
+	                <mesh filename="package://agv_description/meshes/motor_wheel.dae" scale="1.0 1.0 1.0"/>
                 </geometry>
             </collision>
             <inertial>
-                <mass value="1.0" />
+                <mass value="10.0" />
                 <origin xyz="0 0 0" />
-                <inertia  ixx="1.0" ixy="0.0"  ixz="0.0"  iyy="1.0"  iyz="0.0"  izz="1.0" />
+                <inertia  ixx="1.0" ixy="0.0" ixz="0.0"
+                          iyy="1.0" iyz="0.0"
+                          izz="1.0" />
             </inertial>
         </link>
@@ -56,5 +53,7 @@
             <child link="${prefix}_motor_wheel_link"/>
             <axis xyz="0 0 1"/>
-            <limit effort="${steer_joint_effort_limit}" velocity="${steer_joint_velocity_limit}" lower="-1.5708" upper="1.5708"/>
+            <limit effort="${steer_joint_effort_limit}"
+                   velocity="${steer_joint_velocity_limit}"
+                   lower="-1.5708" upper="1.5708"/>
             <joint_properties damping="${steer_joint_damping}" friction="{steer_joint_friction}"/>
         </joint>
@@ -62,8 +61,8 @@
             <type>transmission_interface/SimpleTransmission</type>
             <joint name="${prefix}_motor_wheel_joint">
-                <hardwareInterface>EffortJointInterface</hardwareInterface>
+                <hardwareInterface>hardware_interface/EffortJointInterface</hardwareInterface>
             </joint>
             <actuator name="${prefix}_motor_joint_motor">
-                <hardwareInterface>EffortJointInterface</hardwareInterface>
+                <hardwareInterface>hardware_interface/EffortJointInterface</hardwareInterface>
                 <mechanicalReduction>${motor_wheel_mechanical_reduction}</mechanicalReduction>
             </actuator>
@@ -73,20 +72,22 @@
                 <origin xyz="0 0 0" rpy="0 0 0" />
                 <geometry>
-                    <mesh filename="package://agv_description/meshes/agvs_wheel.dae"/>
+                    <mesh filename="package://agv_description/meshes/agvs_wheel.dae" scale="1.0 1.0 1.0"/>
                 </geometry>
+	            <material name="red">
+	                <color rgba="0.5 0.1 0.1 1"/>
+                </material>
             </visual>
-            <gazebo reference="${prefix}_wheel_link">
-                <material>Gazebo/Gray</material>
-            </gazebo>
             <collision>
                 <origin xyz="0 0 0" rpy="0 0 0" />
                 <geometry>
-	                <mesh filename="package://agv_description/meshes/agvs_wheel.dae"/>
+	                <mesh filename="package://agv_description/meshes/agvs_wheel.dae" scale="1.0 1.0 1.0"/>
                 </geometry>
             </collision>
             <inertial>
-                <mass value="1.250" />
+                <mass value="125.0" />
                 <origin xyz="0 0 0" />
-                <inertia  ixx="1.0" ixy="0.0"  ixz="0.0"  iyy="1.0"  iyz="0.0"  izz="1.0" />
+                <inertia  ixx="1.0" ixy="0.0" ixz="0.0"
+                          iyy="1.0" iyz="0.0"
+                          izz="1.0" />
             </inertial>
         </link>
@@ -102,13 +103,21 @@
             <type>transmission_interface/SimpleTransmission</type>
             <joint name="${prefix}_wheel_joint">
-	            <hardwareInterface>VelocityJointInterface</hardwareInterface>
+	            <hardwareInterface>hardware_interface/VelocityJointInterface</hardwareInterface>
             </joint>
             <actuator name="${prefix}_wheel_joint_motor">
-	            <hardwareInterface>VelocityJointInterface</hardwareInterface>
+	            <hardwareInterface>hardware_interface/VelocityJointInterface</hardwareInterface>
                 <mechanicalReduction>${wheel_mechanical_reduction}</mechanicalReduction>
             </actuator>
         </transmission>
     </xacro:macro>
+    <!-- Macro for agv_base -->
     <xacro:macro name="agv_base">
+        <!--
+        <gazebo>
+            <static>true</static>
+        </gazebo>
+        -->
+        <!-- base_footprint is a fictitious link(frame) that is on the ground right below base_link
+             origin, navigation stack depends on this frame -->
         <link name="base_footprint">
             <visual>
@@ -118,12 +127,7 @@
                 </geometry>
             </visual>
-            <inertial>
-                <mass value="1.250" />
-                <origin xyz="0 0 0" />
-                <inertia  ixx="1.0" ixy="0.0"  ixz="0.0"  iyy="1.0"  iyz="0.0"  izz="1.0" />
-            </inertial>
         </link>
         <joint name="base_footprint_joint" type="fixed">
-            <origin xyz="0 0 0.375" rpy="0 0 0" />
+            <origin xyz="0 0 0.394815" rpy="0 0 0" />
             <parent link="base_footprint"/>
             <child link="base_link" />
@@ -136,8 +140,16 @@
                 </geometry>
             </visual>
+            <collision>
+               <origin xyz="0 0 0" rpy="0 0 0 " />
+               <geometry>
+                    <box size="${base_length} ${base_width} ${base_height}"/>
+               </geometry>
+            </collision>
             <inertial>
-                <mass value="1.250" />
+                <mass value="225.0" />
                 <origin xyz="0 0 0" />
-                <inertia  ixx="1.0" ixy="0.0"  ixz="0.0"  iyy="1.0"  iyz="0.0"  izz="1.0" />
+                <inertia  ixx="1.0" ixy="0.0" ixz="0.0"
+                          iyy="1.0" iyz="0.0"
+                          izz="1.0" />
             </inertial>
         </link>
@@ -145,8 +157,8 @@
             <material>Gazebo/Gray</material>
         </gazebo>
-        <wheel prefix="front_right" x="0.8" y="1.6" z="-0.27"/>
-        <wheel prefix="front_left" x="0.8" y="-1.6" z="-0.27"/>
-        <wheel prefix="back_right" x="-0.8" y="1.6" z="-0.27"/>
-        <wheel prefix="back_left" x="-0.8" y="-1.6" z="-0.27"/>
+        <wheel prefix="front_right" x=" 0.8"  y=" 1.6" z="-0.285"/>
+        <wheel prefix="front_left"  x=" 0.8"  y="-1.6" z="-0.285"/>
+        <wheel prefix="back_right"  x="-0.8"  y=" 1.6" z="-0.285"/>
+        <wheel prefix="back_left"   x="-0.8"  y="-1.6" z="-0.285"/>
     </xacro:macro>
 </robot>

Commit message: Finish_slam_and_add_teleop

File: agv_description/xacro/agv.xacro (robot description, xacro)
@@ -16,9 +16,11 @@
     </joint>
     <xacro:rplidar prefix="laser"/>
-    <!-- property for goods -->
+    <!-- property for goods
     <xacro:property name="goods_offset_x" value="0" />
     <xacro:property name="goods_offset_y" value="0" />
     <xacro:property name="goods_offset_z" value="0.215" />
+-->
     <!-- goods -->
+    <!--
     <joint name="goods_joint" type="fixed">
         <origin xyz="${goods_offset_x} ${goods_offset_y} ${goods_offset_z}" rpy="0 0 0" />
@@ -27,3 +29,4 @@
     </joint>
     <put_7m_goods/>
+    -->
 </robot>

File: agv_description/xacro/agv_base.gazebo.xacro (robot description, xacro)
@@ -1,4 +1,5 @@
 <?xml version="1.0"?>
 <robot>
+<!--
     <gazebo>
         <plugin name="ros_control" filename="libgazebo_ros_control.so">
@@ -8,3 +9,46 @@
         </plugin>
     </gazebo>
+-->
+    <gazebo>
+        <plugin name="agvs_wheel_controller" filename="libgazebo_ros_skid_steer_drive.so">
+            <updateRate>100.0</updateRate>
+            <robotNamespace>/</robotNamespace>
+            <leftFrontJoint>front_left_wheel_joint</leftFrontJoint>
+            <rightFrontJoint>front_right_wheel_joint</rightFrontJoint>
+            <leftRearJoint>back_left_wheel_joint</leftRearJoint>
+            <rightRearJoint>back_right_wheel_joint</rightRearJoint>
+            <wheelSeparation>0.4</wheelSeparation>
+            <wheelDiameter>0.215</wheelDiameter>
+            <robotBaseFrame>base_footprint</robotBaseFrame>
+            <torque>20</torque>
+            <topicName>cmd_vel</topicName>
+            <odometryFrame>odom</odometryFrame>
+            <odometryTopic>odom</odometryTopic>
+            <broadcastTF>true</broadcastTF>
+            <publishTf>true</publishTf>
+            <publishWheelTF>true</publishWheelTF>
+            <publishWheelJointState>true</publishWheelJointState>
+        </plugin>
+    </gazebo>
+    <gazebo>
+        <plugin name="agvs_controller" filename="libgazebo_ros_skid_steer_drive.so">
+            <updateRate>100.0</updateRate>
+            <robotNamespace>/agvs_motor_wheel</robotNamespace>
+            <leftFrontJoint>front_left_motor_wheel_joint</leftFrontJoint>
+            <rightFrontJoint>front_right_motor_wheel_joint</rightFrontJoint>
+            <leftRearJoint>back_left_motor_wheel_joint</leftRearJoint>
+            <rightRearJoint>back_right_motor_wheel_joint</rightRearJoint>
+            <wheelSeparation>0.4</wheelSeparation>
+            <wheelDiameter>0.215</wheelDiameter>
+            <robotBaseFrame>base_footprint</robotBaseFrame>
+            <torque>20</torque>
+            <topicName>cmd_vel</topicName>
+            <odometryFrame>odom</odometryFrame>
+            <odometryTopic>odom</odometryTopic>
+            <broadcastTF>true</broadcastTF>
+            <publishTf>true</publishTf>
+            <publishWheelTF>true</publishWheelTF>
+            <publishWheelJointState>true</publishWheelJointState>
+        </plugin>
+    </gazebo>
 </robot>

File: agv_description/xacro/agv_base.urdf.xacro (robot description, xacro)
@@ -78,8 +78,8 @@
             <type>transmission_interface/SimpleTransmission</type>
             <joint name="${prefix}_motor_wheel_joint">
-                <hardwareInterface>hardware_interface/EffortJointInterface</hardwareInterface>
+                <hardwareInterface>hardware_interface/VelocityJointInterface</hardwareInterface>
             </joint>
             <actuator name="${prefix}_motor_joint_motor">
-                <hardwareInterface>hardware_interface/EffortJointInterface</hardwareInterface>
+                <hardwareInterface>hardware_interface/VelocityJointInterface</hardwareInterface>
                 <mechanicalReduction>${motor_wheel_mechanical_reduction}</mechanicalReduction>
             </actuator>
@@ -162,5 +162,5 @@
             </visual>
         </link>
-        <joint name="base_footprint_joint" type="fixed">
+        <joint name="base_joint" type="fixed">
             <origin xyz="0 0 0.394815" rpy="0 0 0" />
             <parent link="base_footprint"/>

File: agv_description/xacro/sensors/lidar_gazebo.xacro (robot description, xacro)
@@ -56,5 +56,5 @@
                 </ray>
                 <plugin name="gazebo_rplidar" filename="libgazebo_ros_laser.so">
-                    <topicName>/scan</topicName>
+                    <topicName>scan</topicName>
                     <frameName>laser_link</frameName>
                 </plugin>

Commit message: Fix_avoidance_edge_bug

File: agv_description/xacro/agv.xacro (robot description, xacro)
@@ -3,8 +3,14 @@
     <xacro:include filename="$(find agv_description)/xacro/agv_base.urdf.xacro" />
     <xacro:include filename="$(find agv_description)/xacro/sensors/lidar_gazebo.xacro" />
+    <xacro:include filename="$(find agv_description)/xacro/sensors/lidar_gazebo_2.xacro" />
     <xacro:include filename="$(find agv_description)/xacro/goods/goods_gazebo.xacro" />
     <!-- property for lidar -->
-    <xacro:property name="lidar_offset_x" value="0" />
-    <xacro:property name="lidar_offset_y" value="0" />
+    <!--
+    <xacro:property name="lidar_offset_x" value="0.0" />
+    <xacro:property name="lidar_offset_y" value="0.0" />
+    <xacro:property name="lidar_offset_z" value="0.15" />
+    -->
+    <xacro:property name="lidar_offset_x" value="-0.9" />
+    <xacro:property name="lidar_offset_y" value="0.0" />
     <xacro:property name="lidar_offset_z" value="0.15" />
     <agv_base/>
@@ -16,4 +22,15 @@
     </joint>
     <xacro:rplidar prefix="laser"/>
+    <!-- property for lidar -->
+    <xacro:property name="lidar_offset_x_2" value="0.9" />
+    <xacro:property name="lidar_offset_y_2" value="0.0" />
+    <xacro:property name="lidar_offset_z_2" value="0.15" />
+    <!-- lidar2 -->
+    <joint name="lidar_joint_2" type="fixed">
+        <origin xyz="${lidar_offset_x_2} ${lidar_offset_y_2} ${lidar_offset_z_2}" rpy="0 0 0" />
+        <parent link="base_link"/>
+        <child link="laser_2_link"/>
+    </joint>
+    <xacro:rplidar_2 prefix="laser_2"/>
     <!-- property for goods -->
     <xacro:property name="goods_offset_x" value="0" />

File: agv_description/xacro/agv_base.urdf.xacro (robot description, xacro)
@@ -184,8 +184,8 @@
         <wheel prefix="back_left"   x="-0.8"  y="-1.6" z="-0.285"/>
 -->
-        <wheel prefix="front_right" x=" 0.8"  y=" 1.6" z="-0.15"/>
-        <wheel prefix="front_left"  x=" 0.8"  y="-1.6" z="-0.15"/>
-        <wheel prefix="back_right"  x="-0.8"  y=" 1.6" z="-0.15"/>
-        <wheel prefix="back_left"   x="-0.8"  y="-1.6" z="-0.15"/>
+        <wheel prefix="front_right" x=" 0.9"  y=" 1.9" z="-0.15"/>
+        <wheel prefix="front_left"  x=" 0.9"  y="-1.9" z="-0.15"/>
+        <wheel prefix="back_right"  x="-0.9"  y=" 1.9" z="-0.15"/>
+        <wheel prefix="back_left"   x="-0.9"  y="-1.9" z="-0.15"/>
     </xacro:macro>
 </robot>

File: agv_description/xacro/goods/goods_gazebo.xacro (robot description, xacro)
@@ -7,9 +7,9 @@
     <xacro:property name="my_7m_goods_height" value="0.1"/>
     <xacro:property name="my_7m_goods_mass" value="500.0"/>
-    <xacro:property name="legs_length" value="0.15"/>
-    <xacro:property name="legs_width" value="0.15"/>
+    <xacro:property name="legs_length" value="0.05"/>
+    <xacro:property name="legs_width" value="0.125"/>
     <xacro:property name="legs_height" value="0.15"/>
     <xacro:property name="legs_mass" value="10.0"/>
-    <xacro:property name="pillar_radius" value="0.1"/>
+    <xacro:property name="pillar_radius" value="0.05"/>
     <xacro:property name="pillar_width" value="0.05"/>
     <xacro:property name="pillar_mass" value="10.0" />
@@ -111,18 +111,18 @@
         </link>
         <gazebo reference="7m_goods_link">
-            <material>Gazebo/Gray</material>
+            <material>Gazebo/white</material>
         </gazebo>
-        <legs prefix="front_right" x=" 1.175"  y=" 2.925" z="-0.125"/>
-        <legs prefix="front_left"  x=" 1.175"  y="-2.925" z="-0.125"/>
-        <legs prefix="back_right"  x="-1.175"  y=" 2.925" z="-0.125"/>
-        <legs prefix="back_left"   x="-1.175"  y="-2.925" z="-0.125"/>
-        <legs prefix="front_right_2" x=" 1.175"  y=" 2.425" z="-0.125"/>
-        <legs prefix="front_left_2"  x=" 1.175"  y="-2.425" z="-0.125"/>
-        <legs prefix="back_right_2"  x="-1.175"  y=" 2.425" z="-0.125"/>
-        <legs prefix="back_left_2"   x="-1.175"  y="-2.425" z="-0.125"/>
-        <pillar prefix="front_right_2" x=" 0.8"  y=" 1.6" z="-0.075"/>
-        <pillar prefix="front_left_2"  x=" 0.8"  y="-1.6" z="-0.075"/>
-        <pillar prefix="back_right_2"  x="-0.8"  y=" 1.6" z="-0.075"/>
-        <pillar prefix="back_left_2"   x="-0.8"  y="-1.6" z="-0.075"/>
+        <legs prefix="front_right" x=" 1.225"  y=" 3.4375" z="-0.125"/>
+        <legs prefix="front_left"  x=" 1.225"  y="-3.4375" z="-0.125"/>
+        <legs prefix="back_right"  x="-1.225"  y=" 3.4375" z="-0.125"/>
+        <legs prefix="back_left"   x="-1.225"  y="-3.4375" z="-0.125"/>
+        <legs prefix="front_right_2" x=" 1.225"  y=" 2.4375" z="-0.125"/>
+        <legs prefix="front_left_2"  x=" 1.225"  y="-2.4375" z="-0.125"/>
+        <legs prefix="back_right_2"  x="-1.225"  y=" 2.4375" z="-0.125"/>
+        <legs prefix="back_left_2"   x="-1.225"  y="-2.4375" z="-0.125"/>
+        <pillar prefix="front_right_2" x=" 0.9"  y=" 1.9" z="-0.075"/>
+        <pillar prefix="front_left_2"  x=" 0.9"  y="-1.9" z="-0.075"/>
+        <pillar prefix="back_right_2"  x="-0.9"  y=" 1.9" z="-0.075"/>
+        <pillar prefix="back_left_2"   x="-0.9"  y="-1.9" z="-0.075"/>
     </xacro:macro>
 </robot>

File: agv_description/xacro/sensors/lidar_gazebo_2.xacro (robot description, xacro)
@@ -1,7 +1,7 @@
 <?xml version="1.0"?>
-<robot name="laser" xmlns:xacro="http://www.ros.org/wiki/xacro">
+<robot name="laser_2" xmlns:xacro="http://www.ros.org/wiki/xacro">
     <!-- PROPERTY LIST -->
     <xacro:property name="M_PI" value="3.14159265359"/>
-    <xacro:macro name="rplidar" params="prefix:=laser">
+    <xacro:macro name="rplidar_2" params="prefix:=laser">
         <!-- Create laser reference frame -->
         <link name="${prefix}_link">
@@ -31,5 +31,5 @@
         </gazebo>
         <gazebo reference="${prefix}_link">
-            <sensor type="ray" name="rplidar">
+            <sensor type="ray" name="rplidar_2">
                 <pose>0 0 0 0 0 0</pose>
                 <visualize>false</visualize>
@@ -55,7 +55,7 @@
                     </noise>
                 </ray>
-                <plugin name="gazebo_rplidar" filename="libgazebo_ros_laser.so">
-                    <topicName>my_scan</topicName>
-                    <frameName>laser_link</frameName>
+                <plugin name="gazebo_rplidar_2" filename="libgazebo_ros_laser.so">
+                    <topicName>my_scan_2</topicName>
+                    <frameName>laser_2_link</frameName>
                 </plugin>
             </sensor>
